File: single-key-keyboard.kicad_sch (KiCad schematic)
At the start: 27 parts, among them J1 Conn_01x08, J2 Conn_01x05, J5 Conn_01x08, P1 USB_C_Plug_USB2.0, SW1 SW_Push, SW2 SW_SPST, U1 ATtiny416-M

Commit message: Second commit
Parts:
- removed J1, J5: Conn_01x08, Connector_PinSocket_1.00mm:PinSocket_1x08_P1.00mm_Vertical, symbol Connector_Generic:Conn_01x08
- removed TP4: TestPoint, Connector_PinHeader_2.54mm:PinHeader_1x02_P2.54mm_Vertical, symbol Connector:Conn_01x02_Pin
- added TP2: TestPoint, Connector_PinHeader_2.54mm:PinHeader_1x02_P2.54mm_Vertical, symbol Connector:Conn_01x02_Pin
Connections:
- net GND: now also TP3.1 (Pin_1), TP3.2 (Pin_2); no longer SW1.2, TP6.1 (Pin_1), TP6.2 (Pin_2)
- net PA3: now also TP2.1 (Pin_1), TP2.2 (Pin_2); no longer SW1.1, TP1.1 (Pin_1), TP1.2 (Pin_2), TP3.1 (Pin_1), TP3.2 (Pin_2)
- net PA5: no longer D5.2 (A)
- net PB2: now also D5.2 (A)
- new net: SW1.1, TP1.1 (Pin_1), TP1.2 (Pin_2)
- new net GND2: SW1.2, TP6.1 (Pin_1), TP6.2 (Pin_2)
- no-connect marks 3 -> 2
Other:
- moved on the sheet: SW1
