File: single-key-keyboard.kicad_pcb (KiCad board)
At the start: 2 copper layers, 25.4 x 53 mm, 27 parts, among them J1 Conn_01x08, J2 Conn_01x05, J5 Conn_01x08, P1 USB_C_Plug_USB2.0, SW1 SW_Push, SW2 SW_SPST, U1 ATtiny416-M

Commit message: Second commit
Parts:
- removed J1, J5: Conn_01x08, Connector_PinSocket_1.00mm:PinSocket_1x08_P1.00mm_Vertical
- removed TP4: TestPoint, Connector_PinHeader_2.54mm:PinHeader_1x02_P2.54mm_Vertical
- added TP2: TestPoint, Connector_PinHeader_2.54mm:PinHeader_1x02_P2.54mm_Vertical, F.Cu at (130.8, 124.5)
- moved TP3 20.3 mm to (151.1, 124.5)
- moved R3 3.35 mm to (140.5, 119.8), turned to 0 degrees
- moved C1 2.25 mm to (137.4, 123.3), turned to 180 degrees
- moved R4 1.91 mm to (138.9, 121.0), turned to 90 degrees
Connections:
- D5 pad 2: /PA5 -> /PB2
- SW1 pad 1: /PA3 -> Net-(TP1-Pin_1)
- SW1 pad 2: GND -> GND2
- TP1 pad 1: /PA3 -> Net-(TP1-Pin_1)
- TP1 pad 2: /PA3 -> Net-(TP1-Pin_1)
- TP3 pad 1: /PA3 -> GND
- TP3 pad 2: /PA3 -> GND
- TP6 pad 1: GND -> GND2
- TP6 pad 2: GND -> GND2
Routing:
- net /PA3: track 74.7 -> 13.0 mm
- net Net-(TP1-Pin_1): track 0.00 -> 52.8 mm
- net GND2: track 0.00 -> 30.6 mm, vias 0 -> 4
- net GND: track 11.6 -> 35.1 mm, vias 1 -> 4
- net Net-(J2-Pin_5): track 0.00 -> 23.1 mm
- net Net-(J2-Pin_4): track 0.00 -> 15.0 mm
- net +5VP: track 0.00 -> 15.0 mm, vias 0 -> 2
- net /PA4: track 0.00 -> 8.10 mm, vias 0 -> 2
- net /PB2: track 0.00 -> 3.23 mm
- net /PA1 UART TX: track 0.00 -> 1.68 mm
- net /PA2 UART RX: track 0.00 -> 1.37 mm
- net /D-: track 11.3 -> 12.0 mm
- net /PA0 UPDI: track 9.26 -> 9.83 mm
- added copper zone on F.Cu, net GND2
Other:
- outline, holes or cut-outs redrawn

Commit message: Add logo
Parts:
- added G***: LOGO, walking-boat:test7, B.Cu at (143.0, 125.6)
- added H3: MountingHole, panelization:mouse-bite-2.54mm-slot, F.Cu at (127.3, 125.6)
- added H3: MountingHole, panelization:mouse-bite-2.54mm-slot, F.Cu at (127.2, 98.1)
- added H4: MountingHole, panelization:mouse-bite-2.54mm-slot, F.Cu at (141.0, 84.4)
- added REF**: NkJcm501, walking-boat:test, F.Cu at (171.7, 101.1)
Other:
- board size 25.4 x 53 mm -> 30.1 x 57.6 mm
- board text added: "Designed by James Ridey"
